File: PCB/V1/AnalogFaderV1/AnalogFaderV1.sch (KiCad schematic (older format))
At the start: 17 parts, among them J1 USB_B_Micro, SW1 SW_DIP_x03, U1 Opamp_Dual_Generic

Commit message: Added kicad board design files
Added pcb design files for the analog fader V1
Parts:
- removed D1: RED, symbol Device:LED
- removed D2: GREEN, symbol Device:LED
- removed D3: BLUE, symbol Device:LED
- added D1: CLX6F-FKC, digikey-footprints:6-PLCC_3.5x3.5mm, symbol dk_LED-Indication-Discrete:ASMB-TTB0-0A3A2
- added F1: Polyfuse_Small, Fuse_Holders_and_Fuses:Fuse_SMD1206_Wave, symbol Device:Polyfuse_Small
- C1: value C_Small -> 10uf; footprint (none) -> Capacitors_SMD:C_0603
- C2, C3: value C_Small -> 0.1uF; footprint (none) -> Capacitors_SMD:C_0603
- D2: renamed from D4; footprint (none) -> digikey-footprints:SOD-80
- J1: footprint (none) -> 10118194-0001LF:AMPHENOL_10118194-0001LF; symbol Connector:USB_B_Micro -> AnalogFaderV1-rescue:USB_B_Micro-Connector
- R1, R2: value R_Small_US -> 2k; footprint (none) -> Resistors_SMD:R_0603
- R3: value R_Small_US -> 1k; footprint (none) -> Resistors_SMD:R_0603
- R4: value R_Small_US -> 82k; footprint (none) -> Resistors_SMD:R_0603
- R5: value R_Small_US -> 75; footprint (none) -> Resistors_SMD:R_0603
- R6: value R_Small_US -> 105; footprint (none) -> Resistors_SMD:R_0603
- R7: value R_Small_US -> 110 or 63; footprint (none) -> Resistors_SMD:R_0603
- SW1: footprint (none) -> AnalogFaderV1:CVS-03B
- U1: value Opamp_Dual_Generic -> LMV324A; footprint (none) -> digikey-footprints:SOT-23-8
Connections:
- net GND: now also SW1.4, SW1.5, SW1.6
- net VCC: now also F1.2; no longer J1.1 (VBUS)
- net at R7.1: now also SW1.1
- net at R7.2: now also D2.1 (K); no longer SW1.4
- net at R6.1: now also SW1.2
- net at R6.2: now also D1.2; no longer SW1.5
- net at R5.1: now also SW1.3; no longer D2.2 (A)
- net at R5.2: now also D1.1; no longer SW1.6
- new net: D1.4 (R), D1.5 (G), D1.6 (B), U1.6 (-), U1.7
- new net: F1.1, J1.1 (VBUS)
- new net: D1.3, D2.2 (A)
Other:
- note added: "Close to pin"
- note added: "D4 is a diode used to balance the forward voltage of the Red LED (2.1V) \nwith the Blue (3V) and Green (2.7V). The added diode would have a \nforward voltage drop of 0.7V causing the Red LED to turn on around \nthe same time as the Green, and Blue LED"
- note added: "Optional"
- moved on the sheet: C1, C2, C3, D2, J1, R1, R2, R3, R4, R5, R6, R7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

Commit message: Completed Kicad PCB for V1
Finish PCB for V1 of the analog fader circuit.
Parts:
- added R8: 0, symbol Device:R_Small_US
Connections:
- net at D2.1 (K), R7.2: now also R8.1
- net at D1.3, D2.2 (A): now also R8.2
Changed lines of the file:
@@
 	-1   0    0    1
 $EndComp
-Text Notes 2900 3300 0    50   ~ 0
-Optional
-Text Notes 2200 2050 0    50   ~ 0
+Text Notes 2150 1700 0    50   ~ 0
 D4 is a diode used to balance the forward voltage of the Red LED (2.1V) \nwith the Blue (3V) and Green (2.7V). The added diode would have a \nforward voltage drop of 0.7V causing the Red LED to turn on around \nthe same time as the Green, and Blue LED
 Connection ~ 2000 2750
@@
 Connection ~ 2050 2750
 Wire Wire Line
-	3250 2400 3350 2400
+	3250 2400 3300 2400
 $Comp
 L Device:Polyfuse_Small F1
@@
 	2700 2550 2700 2400
 Wire Wire Line
-	2700 2400 2950 2400
+	2700 2400 2900 2400
 Wire Wire Line
 	2700 2950 2700 3100
 Wire Wire Line
 	2700 3100 3350 3100
+Text Notes 2950 2250 0    50   ~ 0
+Optional
+$Comp
+L Device:R_Small_US R8
+U 1 1 600BABD1
+P 3100 2100
+F 0 "R8" V 2895 2100 50  0000 C CNN
+F 1 "0" V 2986 2100 50  0000 C CNN
+F 2 "" H 3100 2100 50  0001 C CNN
+F 3 "~" H 3100 2100 50  0001 C CNN
+	1    3100 2100
+	0    1    1    0
+$EndComp
+Wire Wire Line
+	3200 2100 3300 2100
+Wire Wire Line
+	3300 2100 3300 2400
+Connection ~ 3300 2400
+Wire Wire Line
+	3300 2400 3350 2400
+Wire Wire Line
+	3000 2100 2900 2100
+Wire Wire Line
+	2900 2100 2900 2400
+Connection ~ 2900 2400
+Wire Wire Line
+	2900 2400 2950 2400
 $EndSCHEMATC
