File: Projects/AnalogFadingLED/PCB/V1/AnalogFaderV1/AnalogFaderV1.sch (KiCad schematic (older format))
At the start: 17 parts, among them J1 USB_B_Micro, SW1 SW_DIP_x03, U1 LMV324A

Commit message: Updated PCB to REV 1.1
Fixed inverted footprint for LMV358
Added trace length to switch ground connection for easier soldering
Parts:
- R8: footprint (none) -> Resistors_SMD:R_0603
- U1: value LMV324A -> LMV358; footprint digikey-footprints:SOT-23-8 -> LMV358_sot_23_8:SOT_23_8_LMV358
Changed lines of the file:
@@
 encoding utf-8
 Sheet 1 1
-Title ""
+Title "Analog LED Fader Circuit"
 Date ""
-Rev ""
+Rev "1.1"
 Comp ""
 Comment1 ""
@@
 P 2750 4600
 F 0 "U1" H 2750 4233 50  0000 C CNN
-F 1 "LMV324A" H 2750 4324 50  0000 C CNN
-F 2 "digikey-footprints:SOT-23-8" H 2750 4600 50  0001 C CNN
+F 1 "LMV358" H 2750 4324 50  0000 C CNN
+F 2 "LMV358_sot_23_8:SOT_23_8_LMV358" H 2750 4600 50  0001 C CNN
 F 3 "~" H 2750 4600 50  0001 C CNN
 	1    2750 4600
@@
 P 1650 2750
 F 0 "U1" H 1650 2383 50  0000 C CNN
-F 1 "LMV324A" H 1650 2250 50  0000 C CNN
-F 2 "digikey-footprints:SOT-23-8" H 1650 2750 50  0001 C CNN
+F 1 "LMV358" H 1650 2250 50  0000 C CNN
+F 2 "LMV358_sot_23_8:SOT_23_8_LMV358" H 1650 2750 50  0001 C CNN
 F 3 "~" H 1650 2750 50  0001 C CNN
 	2    1650 2750
@@
 P 5400 2700
 F 0 "U1" H 5358 2746 50  0000 L CNN
-F 1 "LMV324A" V 5150 2350 50  0000 L CNN
-F 2 "digikey-footprints:SOT-23-8" H 5400 2700 50  0001 C CNN
+F 1 "LMV358" V 5150 2350 50  0000 L CNN
+F 2 "LMV358_sot_23_8:SOT_23_8_LMV358" H 5400 2700 50  0001 C CNN
 F 3 "~" H 5400 2700 50  0001 C CNN
 	3    5400 2700
@@
 F 0 "R8" V 2895 2100 50  0000 C CNN
 F 1 "0" V 2986 2100 50  0000 C CNN
-F 2 "" H 3100 2100 50  0001 C CNN
+F 2 "Resistors_SMD:R_0603" H 3100 2100 50  0001 C CNN
 F 3 "~" H 3100 2100 50  0001 C CNN
 	1    3100 2100
